File: Pattern_memo/Adafruit Trellis 4x4 3mm HT16K33.brd (EAGLE design)
At the start: 60 x 60 mm, 42 parts, among them U1 HT16K33 28SOP

Commit message: updated pcb board
Parts:
- removed A0, A1, A2: (no value), microbuilder:SOLDERJUMPER_REFLOW_NOPASTE
- removed C1, C2, C3, C4: (no value), microbuilder:_0805
- removed C5: 10uF, microbuilder:_0805
- removed FID1, FID2, FID3: FIDUCIAL"", microbuilder:FIDUCIAL_1MM
- removed JP1, JP2, JP3, JP4: (no value), microbuilder:1X5_SMT
- removed LED1: TBD, microbuilder:LED3MM-4X4GRID
- removed SW1: (no value), microbuilder:ELAST_PAD_SQUARE_10MM_5.4MM_4X4GRID
- removed TP1, TP2, TP3, TP4: (no value), microbuilder:TESTPOINT_SMT
- removed U$1, U$2: MOUNTINGHOLE2.5, microbuilder:MOUNTINGHOLE_2.5_PLATED
- removed U$3: (no value), microbuilder:ADAFRUIT_TEXT_20MM
- added 5V, ANALOG1, DIGITAL1, DIGITAL2, DIGITAL3, GND: (no value), adafruit:1X01
- added D14, D15, D16, D3: (no value), SparkFun-LED:LED_3MM
- added E$1: (no value), Adafruit Trellis:ELAST_PAD_SQUARE_10MM_5.4MM_4X4GRID
- added R10, R11, R12, R13, R14, R15, R16, R6, R7, R8, R9: 500, SparkFun-Resistors:0603
- added R17, R18, R19, R20, R21, R22, R23, R24, R25, R26, R27, R28, R29, R30, R31, R32: 100, SparkFun-Resistors:0603
- added R33: 100k, SparkFun-Resistors:0603
- added U2: SN74HC595N, SparkFun-IC-Logic:DIP16
- D1, D10, D11, D12, D13, D2, D5, D6, D7, D8, D9: value 1N4148 -> (none); device microbuilder:SOD-323 -> SparkFun-LED:LED_3MM
- D4: value 1N4148 -> (none); device adafruit:SOD-323F -> SparkFun-LED:LED_3MM
- R1, R2: value 10K -> 500; device microbuilder:_0805 -> SparkFun-Resistors:0603
- R3, R4, R5: value 47K -> 500; device rcl:R0805 -> SparkFun-Resistors:0603
- U1: value HT16K33 28SOP -> SN74HC595N; device microbuilder:SOP28_300MIL -> SparkFun-IC-Logic:DIP16
- moved R4 101.5 mm to (75.9, 67.4)
- moved D4 101.2 mm to (73.0, 62.1), flipped to the top
- moved R3 98.2 mm to (63.0, 67.3), turned to 0 degrees
- moved D7 92.7 mm to (58.0, 47.1), flipped to the top
- moved D1 80.4 mm to (28.1, 62.1), flipped to the top
- moved D6 80.2 mm to (43.1, 47.1), flipped to the top, turned to 0 degrees
- moved U1 74.6 mm to (63.1, 39.8)
- moved D11 73.3 mm to (58.0, 32.1), flipped to the top, turned to 0 degrees
- moved D8 71.4 mm to (73.0, 47.1), flipped to the top, turned to 0 degrees
- moved R2 68.7 mm to (46.4, 67.2)
- moved R1 64.6 mm to (32.8, 66.9), turned to 0 degrees
- moved R5 62.6 mm to (23.2, 50.5), turned to 0 degrees
- moved D2 62.2 mm to (43.1, 62.1), flipped to the top, turned to 0 degrees
- moved D10 60.6 mm to (43.1, 32.1), flipped to the top, turned to 0 degrees
- moved D12 56.6 mm to (73.0, 32.1), flipped to the top
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Connections:
- removed net COM0: D4.A, LED1.K13, LED1.K14, LED1.K15, LED1.K16, U1.P$2
- removed net COM1: D1.A, LED1.K10, LED1.K11, LED1.K12, LED1.K9, U1.P$3
- removed net COM2: D2.A, LED1.K5, LED1.K6, LED1.K7, LED1.K8, U1.P$4
- removed net COM3: LED1.K1, LED1.K2, LED1.K3, LED1.K4, U1.P$5
- removed net GND: C1.1, C2.1, C3.1, C4.1, C5.1, JP1.3, JP2.3, JP3.3, JP4.3, U1.P$1
- removed net INT: D13.A, JP1.1, JP2.1, JP3.1, JP4.1
- removed net R0: A2.2, LED1.A9, U1.P$25
- removed net R1: A1.2, LED1.A10, U1.P$24
- removed net R10: LED1.A4, SW1.A4, U1.P$15
- removed net R11: D6.C, D7.C, LED1.A11, U1.P$14
- removed net R12: D10.C, D11.C, LED1.A14, U1.P$13
- removed net R13: LED1.A15, SW1.A15, U1.P$12
- removed net R14: LED1.A16, SW1.A16, U1.P$11
- removed net R2: A0.2, LED1.A13, U1.P$23
- removed net R3: LED1.A6, SW1.A6, U1.P$22
- removed net R4: D12.C, D5.C, LED1.A1, LED1.A5, U1.P$21
- removed net R5: D8.C, D9.C, LED1.A2, U1.P$20
- removed net R6: LED1.A12, SW1.A12, U1.P$19
- removed net R7: LED1.A3, SW1.A3, U1.P$18
- removed net R8: LED1.A8, SW1.A8, U1.P$17
- removed net R9: LED1.A7, SW1.A7, U1.P$16
- removed net SCL: JP1.4, JP2.4, JP3.4, JP4.4, R1.1, U1.P$26
- removed net SDA: JP1.5, JP2.5, JP3.5, JP4.5, R2.2, U1.P$27
- removed net VCC: C1.2, C2.2, C3.2, C4.2, C5.2, JP1.2, JP2.2, JP3.2, JP4.2, R1.2, R2.1, U1.P$28
- new net N$13: D7.K, R7.2
- new net N$14: GND.1, R1.1, R10.1, R11.1, R12.1, R13.1, R14.1, R15.1, R16.1, R2.1, R3.1, R32.2, R4.1, R5.1, R6.1, R7.1, R8.1, R9.1, U1.13, U1.8, U2.13, U2.8
- new net N$15: D8.K, R8.2
- new net N$17: D10.K, R10.2
- new net N$18: D11.K, R11.2
- new net N$21: D14.K, R14.2
- new net N$22: D15.K, R15.2
- new net N$23: D16.K, R16.2
- new net N$24: D1.A, U1.1
- new net N$25: D2.A, U1.2
- new net N$26: D3.A, U1.3
- new net N$27: D4.A, U1.4
- new net N$28: D5.A, U1.5
- new net N$29: D6.A, U1.6
- new net N$30: D7.A, U1.7
- new net N$31: D8.A, U1.15
- new net N$32: D9.A, U2.1
- new net N$33: D10.A, U2.2
- new net N$34: D11.A, U2.3
- new net N$35: 5V.1, R17.1, U1.10, U1.16, U2.10, U2.16
- new net N$36: D12.A, U2.4
- new net N$37: R18.2, R19.1
- new net N$38: D13.A, U2.5
- new net N$39: D14.A, U2.6
- new net N$40: R19.2, R20.1
- new net N$41: D15.A, U2.7
- new net N$42: R20.2, R21.1
- new net N$43: R21.2, R22.1
- new net N$44: R22.2, R23.1
- new net N$45: R23.2, R24.1
- new net N$46: R24.2, R25.1
- new net N$47: R25.2, R26.1
- new net N$48: R26.2, R27.1
- new net N$49: R27.2, R28.1
- new net N$50: R28.2, R29.1
- new net N$51: R29.2, R30.1
- new net N$52: R30.2, R31.1
- new net N$53: R31.2, R32.1
- new net N$54: D16.A, U2.15
- net N$1: now also R17.2, R18.1; no longer D2.C, SW1.B1, SW1.B10, SW1.B13, SW1.B9
- net N$10: now also D4.K, R4.2; no longer D10.A, SW1.A13
- net N$11: now also D5.K, R5.2; no longer D11.A, SW1.A14
- net N$12: now also D6.K, R6.2; no longer D12.A, SW1.A5
- net N$16: now also D9.K, R9.2; no longer D4.C, R3.1, R4.1, R5.1
- net N$19: now also D12.K, R12.2; no longer A1.1, R3.2
- net N$2: now also ANALOG1.1, R33.1; no longer D13.C, U1.P$10
- net N$20: now also D13.K, R13.2; no longer A0.1, R4.2
- net N$3: now also DIGITAL3.1, U1.14; no longer D5.A, SW1.A9
- net N$4: now also DIGITAL1.1, U1.11, U2.11; no longer D6.A, SW1.A10
- net N$5: now also DIGITAL2.1, U1.12, U2.12; no longer D1.C, SW1.B11, SW1.B12, SW1.B14, SW1.B15, SW1.B16, SW1.B2, SW1.B3, SW1.B4, SW1.B5, SW1.B6, SW1.B7, SW1.B8
- net N$6: now also D1.K, R1.2; no longer D7.A, SW1.A11
- net N$7: now also D2.K, R2.2; no longer D8.A, SW1.A1
- net N$8: now also U1.9, U2.14; no longer D9.A, SW1.A2
- net N$9: now also D3.K, R3.2; no longer A2.1, R5.2
Routing:
- net N$5: track 255.9 -> 0.00 mm, vias 1 -> 0
- net SDA: track 215.1 -> 0.00 mm, vias 6 -> 0
- net INT: track 202.8 -> 0.00 mm, vias 6 -> 0
- net SCL: track 193.1 -> 0.00 mm, vias 8 -> 0
- net VCC: track 167.5 -> 0.00 mm, vias 4 -> 0
- net GND: track 162.5 -> 0.00 mm, vias 8 -> 0
- net COM2: track 112.4 -> 0.00 mm, vias 6 -> 0
- net COM1: track 95.2 -> 0.00 mm, vias 4 -> 0
- net COM3: track 84.6 -> 0.00 mm, vias 4 -> 0
- net N$1: track 73.6 -> 0.00 mm, vias 1 -> 0
- net COM0: track 72.6 -> 0.00 mm
- net R4: track 45.5 -> 0.00 mm
- net R12: track 45.5 -> 0.00 mm
- net R2: track 40.5 -> 0.00 mm
- net R14: track 37.9 -> 0.00 mm
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- removed copper zone on layer 16, net VCC
Other:
- board size 60 x 60 mm -> 60.2 x 60.2 mm
- board text removed: "1"
- board text removed: "10"
- board text removed: "11"
- board text removed: "12"
- board text removed: "13"
- board text removed: "14"
- board text removed: "15"
- board text removed: "16"
- board text removed: "2"
- board text removed: "3"
- board text removed: "4"
- board text removed: "4x4 Elastomer Buttons+LEDs"
- board text removed: "5"
- board text removed: "5V"
- board text removed: "6"
- board text removed: "7"
- board text removed: "8"
- board text removed: "9"
- board text removed: "A0"
- board text removed: "A1"
- board text removed: "A2"
- board text removed: "Adafruit Trellis"
- board text removed: "All 3mm LEDs have Anode on left side!"
- board text removed: "GND"
- board text removed: "INT"
- board text removed: "SCL"
- board text removed: "SDA"
- board text removed: "Up to 8 can be tiled when"
- board text removed: "addrs are unique"

Commit message: schematic & board finished
Parts:
- U1, U2: value SN74HC595N -> 74HC595D; device SparkFun-IC-Logic:DIP16 -> Shift_Register:SOT109-1_NXP
- moved R28 73.6 mm to (74.8, 36.6)
- moved R24 70.9 mm to (76.6, 43.6)
- moved R32 70.8 mm to (69.0, 12.7)
- moved R20 65.9 mm to (69.1, 66.5)
- moved R27 60.0 mm to (54.4, 36.6)
- moved R31 59.6 mm to (54.4, 12.6)
- moved R26 57.8 mm to (46.7, 37.1)
- moved R30 55.4 mm to (46.7, 12.8)
- moved R19 50.9 mm to (54.5, 66.7)
- moved R33 48.7 mm to (50.4, 50.0)
- moved R23 47.8 mm to (54.1, 42.3)
- moved R29 47.5 mm to (32.1, 13.5)
- moved R18 42.9 mm to (47.2, 66.9)
- moved R22 40.0 mm to (46.9, 42.5)
- moved R25 40.0 mm to (24.5, 36.1)
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Connections:
- removed net N$28 (its old number): D5.A, U1.5
- removed net N$34: D11.A, U2.3
- new net N$4: D11.A, U2.2
- new net N$8: GND.1, R1.1, R10.1, R11.1, R12.1, R13.1, R14.1, R15.1, R16.1, R2.1, R3.1, R32.2, R33.2, R4.1, R5.1, R6.1, R7.1, R8.1, R9.1, U1.13, U1.8, U2.13, U2.8
- net N$14: now also D1.A, U1.15; no longer GND.1, R1.1, R10.1, R11.1, R12.1, R13.1, R14.1, R15.1, R16.1, R2.1, R3.1, R32.2, R4.1, R5.1, R6.1, R7.1, R8.1, R9.1, U1.13, U1.8, U2.13, U2.8
- net N$24: now also D5.A, U1.4; no longer D1.A, U1.1
- net N$25: now also U1.1; no longer U1.2
- net N$26: now also U1.2; no longer U1.3
- net N$27: now also U1.3; no longer U1.4
- net N$29: now also U1.5; no longer U1.6
- net N$30: now also U1.6; no longer U1.7
- net N$31: now also U1.7; no longer U1.15
- net N$32: now also D13.A, U2.4; no longer D9.A, U2.1
- net N$33: now also U2.1; no longer U2.2
- net N$36: now also U2.3; no longer U2.4
- net N$38: now also D9.A, U2.15; no longer D13.A, U2.5
- net N$39: now also U2.5; no longer U2.6
- net N$41: now also U2.6; no longer U2.7
- net N$54: now also U2.7; no longer U2.15
Routing:
- net N$2: track 0.00 -> 409.4 mm, vias 0 -> 13
- net N$35: track 0.00 -> 170.0 mm, vias 0 -> 10
- net N$43: track 0.00 -> 150.0 mm, vias 0 -> 5
- net N$55: track 0.00 -> 112.6 mm, vias 0 -> 9
- net N$28: track 0.00 -> 109.8 mm, vias 0 -> 4
- net N$46: track 0.00 -> 99.6 mm, vias 0 -> 3
- net N$5: track 0.00 -> 98.1 mm, vias 0 -> 4
- net N$50: track 0.00 -> 66.9 mm, vias 0 -> 3
- net N$47: track 0.00 -> 61.1 mm, vias 0 -> 3
- net N$3: track 0.00 -> 59.3 mm, vias 0 -> 2
- net N$45: track 0.00 -> 58.7 mm, vias 0 -> 5
- net N$42: track 0.00 -> 55.9 mm, vias 0 -> 3
- net N$24: track 0.00 -> 52.8 mm, vias 0 -> 2
- net N$14: track 0.00 -> 51.7 mm, vias 0 -> 4
- net N$54: track 0.00 -> 48.6 mm, vias 0 -> 2
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- added copper zone on layer 16, net N$8
Other:
- board text added: "NL + GG"
- board text added: "SPARK HACK IT"

Commit message: fixed errors in PCB board
Parts:
- moved DIGITAL3 0.25 mm to (65.5, 21.3)
Routing:
- net N$8: track 1.28 -> 17.6 mm, vias 0 -> 2
- net N$3: track 59.3 -> 75.4 mm
- net N$25: track 30.6 -> 36.1 mm
- net N$2: track 409.4 -> 414.7 mm
- net N$35: track 170.0 -> 165.6 mm, vias 10 -> 12
- net N$43: track 150.0 -> 154.2 mm
- net N$55: track 112.6 -> 116.1 mm
- net N$12: track 23.5 -> 26.6 mm
- net N$39: track 35.7 -> 38.7 mm
- net N$1: track 23.7 -> 26.2 mm
- net N$33: track 20.0 -> 21.9 mm
- net N$44: track 16.6 -> 18.4 mm
- net N$5: track 98.1 -> 99.7 mm
- net N$45: track 58.7 -> 60.2 mm
- net N$37: track 25.4 -> 26.6 mm
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Other:
- board text added: "NL + GG Dec 2022"
- board text removed: "NL + GG"
